Commit message: 更新urdf

File: legged_gym/resources/robots/mybot_v3/urdf/mybot_v3.urdf (robot description, URDF)
Before this commit: robot mybot_v3, 19 links, 18 joints
Links:
- removed link payload_link
- link FL_calf: mass 0.23708419 -> 0.23880158
- link FR_calf: mass 0.23765586 -> 0.23880158
Joints:
- removed joint payload_joint

Commit message: Update mybot_v3 inertial properties

File: legged_gym/resources/robots/mybot_v3/urdf/mybot_v3.urdf (robot description, URDF)
Before this commit: robot mybot_v3, 18 links, 17 joints
Links:
- link FL_calf: mass 0.23880158 -> 0.23708419
- link FR_calf: mass 0.23880158 -> 0.23708419
- link RR_thigh: mass 1.42118841 -> 1.45068546

Commit message: Update mybot_v3 inertial properties from revised data

File: legged_gym/resources/robots/mybot_v3/urdf/mybot_v3.urdf (robot description, URDF)
Before this commit: robot mybot_v3, 18 links, 17 joints
Links:
- link FL_thigh: mass 1.44059854 -> 1.42386939
- link FR_thigh: mass 1.44059854 -> 1.42386939
- link RL_thigh: mass 1.45185979 -> 1.43392711
- link RR_calf: mass 0.23880158 -> 0.22489484
- link RR_thigh: mass 1.45068546 -> 1.40325573
